File: hardware/lidarlite-hat.kicad_pcb (KiCad board)
At the start: 4 copper layers, 0 parts

Commit message: In progress. Just playing around.
Parts:
- added C1: 100nF, Wickerlib:0402, F.Cu at (138.2, 98.6)
- added C10: 100nF 10V, Wickerlib:0402, F.Cu at (109.2, 105.1)
- added C11: 100nF 10V, Wickerlib:0402, F.Cu at (124.6, 102.7)
- added C2: 100nF 10V, Wickerlib:0402, F.Cu at (136.1, 94.6)
- added C3: 1uF 25V, Wickerlib:0603, F.Cu at (113.4, 90.9)
- added C4: 1uF 25V, Wickerlib:0603, F.Cu at (119.0, 87.2)
- added C5: 100nF 10V, Wickerlib:0402, F.Cu at (137.2, 104.2)
- added C6: 1uF 25V, Wickerlib:0603, F.Cu at (134.7, 104.8)
- added C7: 22pF, Wickerlib:0603, F.Cu at (114.2, 106.9)
- added C8: 22pF, Wickerlib:0603, F.Cu at (125.0, 108.9)
- added C9: 100nF 10V, Wickerlib:0402, F.Cu at (120.6, 91.0)
- added D1: 20V 1A, Wickerlib:Diode_SMA, F.Cu at (104.9, 87.2)
- added F1: 500mA, 1812, F.Cu at (108.3, 91.4)
- added J1: MICRO-SD, Wickerlib:Conn_uSDcard, F.Cu at (150.9, 96.7)
- added J2: USB-MICROB-10118193, Wickerlib:USB-Micro-B-10118193_0001LF, F.Cu at (100.8, 97.3)
- added J3: ICSP, Wickerlib:Pin_Header_Straight_2x03, F.Cu at (132.9, 88.5)
- added J4: LIDAR, Wickerlib:Pin_Header_Straight_1x06, F.Cu at (117.7, 114.3)
- added L1: FERRITE, Wickerlib:0402, F.Cu at (107.4, 100.1)
- added LED1: RED, Wickerlib:0603, F.Cu at (122.9, 89.8)
- added P7: CONN_1, Wickerlib:ARDUINO-MOUNTING-HOLE, F.Cu at (142.2, 111.3)
- added P7: CONN_1, Wickerlib:ARDUINO-MOUNTING-HOLE, F.Cu at (111.8, 111.3)
- added P7: CONN_1, Wickerlib:ARDUINO-MOUNTING-HOLE, F.Cu at (142.2, 83.8)
- added P7: CONN_1, Wickerlib:ARDUINO-MOUNTING-HOLE, F.Cu at (111.8, 83.8)
- added R1: 1K, Wickerlib:0603, F.Cu at (122.3, 87.2)
- added R2: 22, 0603, F.Cu at (107.3, 96.0)
- added R3: 22, 0603, F.Cu at (107.4, 97.8)
- added R4: 10K, 0603, F.Cu at (106.6, 104.5)
- added S1: RESET, Wickerlib:SW-B3U-1000P, F.Cu at (104.4, 107.0)
- added U1: MAX3377, Wickerlib:TSSOP-14_4.4x5mm_Pitch0.65mm, F.Cu at (133.6, 99.5)
- added U2: MIC5365, Wickerlib:SOT-23-5, F.Cu at (117.2, 90.0)
- added U3: IC-MCU-ATMEGA32U4-TQFP44, Wickerlib:TQFP-44_10x10mm_Pitch0.8mm, F.Cu at (116.8, 99.0)
- added X1: 16MHZ, Wickerlib:CRYSTAL-CTS-4SMD, F.Cu at (122.9, 107.3)
Routing:
- net +5V: track 0.00 -> 99.9 mm, vias 0 -> 6
- net GND: track 0.00 -> 60.7 mm, vias 0 -> 15
- net /MISO: track 0.00 -> 39.5 mm, vias 0 -> 2
- net /SCLK: track 0.00 -> 37.9 mm, vias 0 -> 2
- net +3V3: track 0.00 -> 37.2 mm, vias 0 -> 4
- net /~RESET: track 0.00 -> 35.9 mm, vias 0 -> 2
- net /MOSI: track 0.00 -> 35.8 mm, vias 0 -> 2
- net /CS: track 0.00 -> 24.2 mm, vias 0 -> 2
- net /LIDAR_MODE: track 0.00 -> 20.7 mm, vias 0 -> 1
- net /SCL: track 0.00 -> 20.0 mm, vias 0 -> 1
- net /LIDAR_EN: track 0.00 -> 18.6 mm, vias 0 -> 1
- net /SD_MISO: track 0.00 -> 18.4 mm, vias 0 -> 2
- net /SDA: track 0.00 -> 17.4 mm, vias 0 -> 1
- net /VUSB_IN: track 0.00 -> 15.0 mm
- net /~3STATE: track 0.00 -> 13.4 mm, vias 0 -> 2
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Other:
- board outline added: 48.3 x 34.4 mm
- copper layers 4 -> 2
