File: hardware/lidarlite-hat.sch (KiCad schematic (older format))
At the start: 0 parts

Commit message: Added microSD circuit.
Parts:
- added J?: MICRO-SD, SD-5009010801, symbol CONN-MICRO-SD-CARD-PUSH-PULL
Connections:
- net labels added: +3.3V, GND, SD_CS, SD_MISO, SD_MOSI, SD_SCLK
- wire segments 0 -> 8
Changed lines of the file:
@@
 Comment4 ""
 $EndDescr
+$Comp
+L CONN-MICRO-SD-CARD-PUSH-PULL J?
+U 1 1 577E0D25
+P 5500 2650
+F 0 "J?" H 5100 3250 50  0000 L CNN
+F 1 "MICRO-SD" H 5100 2050 50  0000 L CNN
+F 2 "SD-5009010801" H 5500 2300 50  0001 C CIN
+F 3 "http://www.molex.com/pdm_docs/sd/5009010801_sd.pdf" H 5500 2650 5   0001 C CNN
+F 4 "UNDEFINED" H 5500 2300 50  0001 C CIN "Package"
+F 5 "Molex" H 5500 2300 50  0001 C CIN "MF_Name"
+F 6 "5009010801" H 5500 2300 50  0001 C CIN "MF_PN"
+F 7 "Digikey" H 5500 2300 50  0001 C CIN "S1_Name"
+F 8 "WM19081CT-ND" H 5500 2300 50  0001 C CIN "S1_PN"
+F 9 "CONN MICRO SD CARD HINGED TYPE" H 5500 2300 50  0001 C CIN "Description"
+F 10 "Not Verified" H 5500 2300 50  0001 C CIN "Verified"
+	1    5500 2650
+	1    0    0    -1
+$EndComp
+Wire Wire Line
+	4900 2200 4375 2200
+Wire Wire Line
+	4375 2300 4900 2300
+Wire Wire Line
+	4900 2400 4375 2400
+Wire Wire Line
+	4900 2500 4375 2500
+Wire Wire Line
+	4900 3000 4700 3000
+Wire Wire Line
+	4700 3000 4700 2900
+Wire Wire Line
+	4900 3100 4700 3100
+Wire Wire Line
+	4700 3100 4700 3175
+$Comp
+L GND #PWR?
+U 1 1 577E0DED
+P 4700 3175
+F 0 "#PWR?" H 4700 2925 50  0001 C CNN
+F 1 "GND" H 4700 3025 50  0000 C CNN
+F 2 "" H 4700 3175 50  0000 C CNN
+F 3 "" H 4700 3175 50  0000 C CNN
+	1    4700 3175
+	1    0    0    -1
+$EndComp
+$Comp
+L +3.3V #PWR?
+U 1 1 577E0E03
+P 4700 2900
+F 0 "#PWR?" H 4700 2750 50  0001 C CNN
+F 1 "+3.3V" H 4700 3040 50  0000 C CNN
+F 2 "" H 4700 2900 50  0000 C CNN
+F 3 "" H 4700 2900 50  0000 C CNN
+	1    4700 2900
+	1    0    0    -1
+$EndComp
+Text Label 4475 2200 0    60   ~ 0
+SD_MOSI
+Text Label 4475 2300 0    60   ~ 0
+SD_MISO
+Text Label 4475 2400 0    60   ~ 0
+SD_SCLK
+Text Label 4475 2500 0    60   ~ 0
+SD_CS
 $EndSCHEMATC

Commit message: In progress. Just playing around.
Parts:
- added C1: 100nF, Wickerlib:0402, symbol CAP-CER-100NF-10V-X7R-0402
- added C10, C11, C2, C5, C9: 100nF 10V, Wickerlib:0402, symbol CAP-CER-100NF-10V-X7R-0402
- added C3, C4, C6: 1uF 25V, Wickerlib:0603, symbol CAP-CER-1UF-25V-X7R-0603
- added C7, C8: 22pF, Wickerlib:0603, symbol CAP-CER-22PF-100V-C0G-NP0-0603
- added D1: 20V 1A, Wickerlib:Diode_SMA, symbol DIODE-SCHOTTKY-20V-1A-SS12-SMA
- added F1: 500mA, Wickerlib:1812, symbol FUSE-RESET-500MA-15V-MF-MSMF
- added J2: USB-MICROB-10118193, Wickerlib:USB-Micro-B-10118193_0001LF, symbol CONN-USB-MICRO-B-10118193
- added J3: ICSP, Wickerlib:Pin_Header_Straight_2x03, symbol HEADER-MALE-6POS-TH-2x3-P0.1IN
- added J4: LIDAR, Wickerlib:Pin_Header_Straight_1x06, symbol HEADER-FEMALE-6POS-TH-1x06-P0.1IN
- added J?: KEYPAD, CONN-1x07-2.54MM-TH, symbol HEADER-FEMALE-7POS-TH-1x07-P0.1IN
- added L1: FERRITE, Wickerlib:0402, symbol FERRITE-BEAD-220-OHM-0402-1LN
- added LED1: RED, Wickerlib:0603, symbol LED-RED-0603-SMT-HSMS-C191
- added R1: 1K, Wickerlib:0603, symbol RES-1K-1%-1/10W-0603
- added R2, R3: 22, Wickerlib:0603, symbol RES-22-OHM-5%-1/10W-0603
- added R4: 10K, Wickerlib:0603, symbol RES-10K-1%-1/8W-0603
- added S1: RESET, Wickerlib:SW-B3U-1000P, symbol SWITCH-TACTILE-SPST-NO-0.05A-12V
- added U1: MAX3377, Wickerlib:TSSOP-14_4.4x5mm_Pitch0.65mm, symbol IC-LEVEL-TRANS-MAX3377-TSSOP14
- added U2: MIC5365, Wickerlib:SOT-23-5, symbol IC-REG-LDO-3.3V-0.5A-BU33SD5WG-SSOP5
- added U3: IC-MCU-ATMEGA32U4-TQFP44, Wickerlib:TQFP-44_10x10mm_Pitch0.8mm, symbol IC-MCU-ATMEGA32U4-TQFP44
- added X1: 16MHZ, Wickerlib:CRYSTAL-CTS-4SMD, symbol CRYSTAL-16MHZ-18PF-40OHM-CTS-4SMD
- J1: renamed from J?; footprint SD-5009010801 -> Wickerlib:Conn_uSDcard
Connections:
- net labels added: +5V, CS, HEARTBEAT, LIDAR_EN, LIDAR_MODE, MISO, MOSI, SCL, SCLK, SDA, UGND, USB_D+, USB_D-, VUSB, VUSB_IN, ~3STATE, ~RESET
- wire segments 8 -> 110
Other:
- note added: "3.3V - 5V\nLEVEL TRANSLATE"
- note added: "LDO\n"
- note added: "TODO: SPEAKER\nKEYPAD\nPAUSE BUTTON"
- moved on the sheet: J1

Commit message: Some hardware adds.
Parts:
- removed D1: 20V 1A, Wickerlib:Diode_SMA, symbol DIODE-SCHOTTKY-20V-1A-SS12-SMA
- removed U1: MAX3377, Wickerlib:TSSOP-14_4.4x5mm_Pitch0.65mm, symbol IC-LEVEL-TRANS-MAX3377-TSSOP14
- removed U2: MIC5365, Wickerlib:SOT-23-5, symbol IC-REG-LDO-3.3V-0.5A-BU33SD5WG-SSOP5
- added C12: 1uF, 0603, symbol CAP-CER-1UF-25V-X7R-0603
- added D2, D3: CG0603MLC-05E, 0603, symbol DIODE-TVS-CG0603MLC-05E
- added D?: 20V 1A, Diode_SMA, symbol DIODE-SCHOTTKY-20V-B120-13-F-1A-SMA
- added J5: ON/OFF, CONN-1x02-2.54MM-TH, symbol HEADER-MALE-2POS-TH-1x02-P0.1IN
- added Q1: MMBT3904, SOT23-3, symbol BJT-NPN-40V-0.2A-MMBT3904
- added R5: 220, 0603, symbol RES-220-5%-1/10W-0603
- added R6: 10, 0603, symbol RES-10-1%-1/10W-0603
- added SPK1: 8OHM, PSR-2WIRE, symbol SPEAKER-8OHM-23MM-ROUND-2PIN
- added U?: MAX3377, TSSOP14, symbol IC-LEVEL-TRANS-MAX3377-TSSOP14
- added U?: MCP1703, SOT23A-3, symbol IC-REG-LDO-3.3V-0.25A-MCP1703-SOT23A-3
- C7: MF_PN C0805C220J5GACTU -> C0603C220J1GACTU
- gave numbers to parts that had none: 1
Connections:
- net +3V3: now also U?.1 (VL), U?.2 (OUT)
- net +5V: now also D?.1 (K), R6.1, U?.14 (VCC), U?.3 (IN)
- net CS: now also U?.10 (IOVCC4)
- net GND: now also D2.2, D3.2, Q1.2 (E), SPK1.2, U?.1 (GND), U?.7 (GND)
- net MISO: now also U?.12 (IOVCC2)
- net MOSI: now also U?.13 (IOVCC1)
- net SCLK: now also U?.11 (IOVCC3)
- net SD_CS: now also U?.5 (IOVL4)
- net SD_MISO: now also U?.3 (IOVL2)
- net SD_MOSI: now also U?.2 (IOVL1)
- net SD_SCLK: now also U?.4 (IOVL3)
- net VUSB: now also D?.2 (A)
- net ~3STATE: now also U?.8 (~3STATE)
- net at J2.2 (D-), R2.2: now also D2.1
- net at J2.3 (D+), R3.2: now also D3.1
- new net: C12.1, SPK1.1
- new net: C12.2, Q1.3 (C), R6.2
- new net: Q1.1 (B), R5.1
- new net SPK_PWM: R5.2
Other:
- note removed: "TODO: SPEAKER\nKEYPAD\nPAUSE BUTTON"
- moved on the sheet: C1, C10, C11, C2, C3, C4, C5, C6, C7, C8, C9, F1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
